Commit message: added manipulator to tbot and some cleanup

File: open_manipulator_x_description/gazebo/materials.xacro (robot description, xacro)
@@ -14,7 +14,8 @@
     <color rgba="0.8706 0.8118 0.7647 1.0"/>
   </material>
+<!--
   <material name="dark">
     <color rgba="0.3 0.3 0.3 1.0"/>
-  </material>
+  </material> -->
   <material name="green">
     <color rgba="0.0 0.8 0.0 1.0"/>
@@ -23,7 +24,7 @@
     <color rgba="0.5 0.5 0.5 1.0"/>
   </material>
-  <material name="light_black">
+  <!-- <material name="light_black">
     <color rgba="0.4 0.4 0.4 1.0"/>
-  </material>
+  </material> -->
   <material name="orange">
     <color rgba="1.0 0.4235 0.0392 1.0"/>

File: open_manipulator_x_description/urdf/open_manipulator_x_robot.urdf.xacro (robot description, xacro)
@@ -3,8 +3,4 @@
 <robot name="open_manipulator_x" xmlns:xacro="http://ros.org/wiki/xacro">
   <xacro:arg name="prefix" default="" />
-  <xacro:arg name="use_sim" default="false" />
-  <xacro:arg name="use_fake_hardware" default="false" />
-  <xacro:arg name="fake_sensor_commands" default="false" />
-  <xacro:arg name="port_name" default="/dev/ttyUSB0" />
   <!-- Import Rviz colors -->
   <xacro:include filename="$(find open_manipulator_x_description)/gazebo/materials.xacro" />
@@ -20,7 +16,4 @@
   <xacro:open_manipulator_x_gazebo prefix="$(arg prefix)" />
   <gazebo>
-    <!-- <plugin name="gazebo_ros2_control" filename="libgazebo_ros2_control.so">
-      <parameters>$(find open_manipulator_x_bringup)/config/gazebo_controller_manager.yaml</parameters>
-    </plugin> -->
     <plugin filename="gz_ros2_control-system" name="gz_ros2_control::GazeboSimROS2ControlPlugin">
       <robot_param>robot_description</robot_param>
@@ -29,9 +22,4 @@
     </plugin>
   </gazebo>
-  <!-- <xacro:open_manipulator_x_system
-    name="OpenManipulatorXSystem" prefix="$(arg prefix)" use_sim="$(arg use_sim)"
-    use_fake_hardware="$(arg use_fake_hardware)"
-    fake_sensor_commands="$(arg fake_sensor_commands)"
-    port_name="$(arg port_name)" /> -->
   <xacro:open_manipulator_x_system name="OpenManipulatorXSystem" prefix="$(arg prefix)" />
   <!-- World -->
